File: hw/synthopl/synthopl.kicad_sch (KiCad schematic)
At the start: 21 parts, among them J2 AudioJack3, U1 6N137, U2 74HC595, U3 NE5532, U4 NE5532, U5 74HCT245, U6 YMF262-M, U7 YAC512-M, X1 14.318MHz

Commit message: fixes
Parts:
- removed J2: AudioJack3, Connector_Audio:Jack_3.5mm_Lumberg_1503_07_Horizontal, symbol Connector_Audio:AudioJack3
- removed R3, R4: 10k, symbol Device:R
- added C10, C11, C12, C14, C15, C7, C8, C9: 100nF, symbol Device:C
Connections:
- net +3V3: now also U5.9 (A7), C7.1
- net +5V: now also C10.1, C12.1, C14.1, C15.1, C9.1; no longer U6.7 (RD)
- net +9V: now also C11.1, C8.1
- net GNDA: now also C10.2, C11.2, C12.2, C14.2, C15.2, C7.2, C8.2, C9.2
- net at U5.11 (B7): now also U6.7 (RD)
- net MIDI_A: now reaches R1.2
- net at U2.7 (QH), U6.18 (D7): no longer U6.20 (SMPAC), U7.8 (SMP1)
- net MIDI_K: now reaches D1.2 (A), U1.3 (C)
- new net SMP1: U6.20 (SMPAC), U7.8 (SMP1)
- no-connect marks 9 -> 8
Other:
- moved on the sheet: U3C, U4C, U7

Commit message: add opl3 footprint
Parts:
- R2: footprint (none) -> Resistor_THT:R_Axial_DIN0204_L3.6mm_D1.6mm_P5.08mm_Horizontal
- U6: footprint Package_SO:SOP-24_7.5x15.4mm_P1.27mm -> OPL3:SOIC-24W_8.5
Changed lines of the file:
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@@
       (effects (font (size 1.27 1.27)))
     )
-    (property "Footprint" "Package_SO:SOP-24_7.5x15.4mm_P1.27mm" (at 95.25 128.27 0)
+    (property "Footprint" "OPL3:SOIC-24W_8.5" (at 95.25 128.27 0)
       (effects (font (size 1.27 1.27)) hide)
     )
@@
       (effects (font (size 1.27 1.27)) (justify left))
     )
-    (property "Footprint" "" (at 83.312 29.21 90)
-      (effects (font (size 1.27 1.27)) hide)
-    )
+    (property "Footprint" "Resistor_THT:R_Axial_DIN0204_L3.6mm_D1.6mm_P5.08mm_Horizontal" (at 83.312 29.21 90)
+      (effects (font (size 1.27 1.27)) hide)
+    )

Commit message: switch L/R channels
Connections:
- net LEFT: now also C6.2; no longer C5.2
- net RIGHT: now also C5.2; no longer C6.2
Changed lines of the file:
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@@
     )
   )
-  (global_label "RIGHT" (shape output) (at 274.32 149.86 0) (fields_autoplaced)
+  (global_label "LEFT" (shape output) (at 274.32 149.86 0) (fields_autoplaced)
     (effects (font (size 1.27 1.27)) (justify left))
-    (property "Intersheetrefs" "${INTERSHEET_REFS}" (at 282.7481 149.86 0)
+    (property "Intersheetrefs" "${INTERSHEET_REFS}" (at 281.5385 149.86 0)
       (effects (font (size 1.27 1.27)) (justify left) hide)
     )
@@
     )
   )
-  (global_label "LEFT" (shape output) (at 274.32 123.19 0) (fields_autoplaced)
+  (global_label "RIGHT" (shape output) (at 274.32 123.19 0) (fields_autoplaced)
     (effects (font (size 1.27 1.27)) (justify left))
-    (property "Intersheetrefs" "${INTERSHEET_REFS}" (at 281.5385 123.19 0)
+    (property "Intersheetrefs" "${INTERSHEET_REFS}" (at 282.7481 123.19 0)
       (effects (font (size 1.27 1.27)) (justify left) hide)
     )
